Commit message: model complate

File: description/robot_model.xacro (robot description, xacro)
@@ -14,8 +14,11 @@
         <color rgba="0 0 0 1"/>
     </material>
+    <material name="red">
+        <color rgba="1 0 0 1"/>
+    </material>
     <!-- BASE_FOOTPRINT LINK-->
     <joint name="base_footprint_joint" type="fixed">
-        <parent link="base_link"/>
-        <child link="base_footprint"/>
+        <parent link="base_footprint"/>
+        <child link="base_link"/>
         <origin xyz="0 0 0" rpy="0 0 0"/>
     </joint>
@@ -24,26 +27,26 @@
     <link name="base_link">
         <visual>
-            <origin xyz="-0.1 0 0.1" rpy="0 0 0"/>
+            <origin xyz="0.0 0.0 0.0" rpy="0 0 0"/>
             <geometry>
-                <box size="0.2 0.50 0.2"/>
+                <box size="0.175 0.110 0.07975"/>
             </geometry>
             <material name="black"/>
         </visual>
         <collision>
-            <origin xyz="-0.1 0 0.1" rpy="0 0 0"/>
+            <origin xyz="0.0 0.0 0.0" rpy="0 0 0"/>
             <geometry>
-                <box size="0.2 0.50 0.2"/>
+                <box size="0.175 0.110 0.07975"/>
             </geometry>
             <material name="black"/>
         </collision>
-        <xacro:inertial_box mass="2.0" x="0.2" y="0.50" z="0.2">
-            <origin xyz="-0.1 0 0.1" rpy="0 0 0"/>
+        <xacro:inertial_box mass="0.5" x="0.175" y="0.110" z="0.07975">
+            <origin xyz="0.0 0.0 0.0" rpy="0 0 0"/>
         </xacro:inertial_box>
     </link>
     <!-- Tekerlekler -->
-    <link name="fork_left_wheel">
+    <link name="left_wheel">
         <visual>
             <geometry>
-                <cylinder radius="0.03" length="0.02"/>
+                <cylinder radius="0.0325" length="0.03"/>
             </geometry>
             <material name="orange"/>
@@ -51,16 +54,16 @@
         <collision>
             <geometry>
-                <cylinder radius="0.03" length="0.02"/>
+                <cylinder radius="0.0325" length="0.03"/>
             </geometry>
             <material name="orange"/>
         </collision>
-        <xacro:inertial_cylinder mass="0.1" length="0.02" radius="0.03">
+        <xacro:inertial_cylinder mass="0.1" length="0.03" radius="0.0325">
             <origin xyz="0 0 0" rpy="0 0 0"/>
         </xacro:inertial_cylinder>
     </link>
-    <link name="fork_right_wheel">
+    <link name="right_wheel">
         <visual>
             <geometry>
-                <cylinder radius="0.03" length="0.02"/>
+                <cylinder radius="0.0325" length="0.03"/>
             </geometry>
             <material name="orange"/>
@@ -68,121 +71,47 @@
         <collision>
             <geometry>
-                <cylinder radius="0.03" length="0.02"/>
+                <cylinder radius="0.0325" length="0.03"/>
             </geometry>
             <material name="orange"/>
         </collision>
-        <xacro:inertial_cylinder mass="0.1" length="0.02" radius="0.03">
+        <xacro:inertial_cylinder mass="0.1" length="0.03" radius="0.0325">
             <origin xyz="0 0 0" rpy="0 0 0"/>
         </xacro:inertial_cylinder>
     </link>
-    <link name="front_wheel">
+    <link name="caster_wheel">
         <visual>
             <geometry>
-                <cylinder radius="0.07" length="0.04"/>
+                <sphere radius="0.015" />
             </geometry>
-            <material name="orange"/>
+            <material name="red"/>
         </visual>
         <collision>
             <geometry>
-                <cylinder radius="0.07" length="0.04"/>
+                <sphere radius="0.05"/>
             </geometry>
-            <material name="orange"/>
+            <material name="red"/>
         </collision>
-        <xacro:inertial_cylinder mass="0.1" length="0.04" radius="0.07">
+        <xacro:inertial_sphere mass="0.15" radius="0.05">
             <origin xyz="0 0 0" rpy="0 0 0"/>
-        </xacro:inertial_cylinder>
-    </link>
-    <!-- Direksyon Mekanizması -->
-    <link name="steering_cylinder">
-        <visual>
-            <geometry>
-                <cylinder radius="0.01" length="0.2"/>
-            </geometry>
-            <material name="blue"/>
-        </visual>
-        <collision>
-            <geometry>
-                <cylinder radius="0.01" length="0.2"/>
-            </geometry>
-            <material name="blue"/>
-        </collision>
-        <xacro:inertial_cylinder mass="0.1" length="0.2" radius="0.01">
-            <origin xyz="0 0 0" rpy="0 0 0"/>
-        </xacro:inertial_cylinder>
-    </link>
-    <!-- Çatal Mekanizması -->
-    <link name="left_fork">
-        <visual>
-            <origin xyz="0.575 0 0.025"/>
-            <geometry>
-                <box size="1.15 0.14 0.05"/>
-            </geometry>
-            <material name="white"/>
-        </visual>
-        <collision>
-            <origin xyz="0.575 0 0.025"/>
-            <geometry>
-                <box size="1.15 0.14 0.05"/>
-            </geometry>
-            <material name="white"/>
-        </collision>
-        <xacro:inertial_box mass="5.0" x="1.14" y="0.14" z="0.05">
-            <origin xyz="0.575 0 0.025" rpy="0 0 0"/>
-        </xacro:inertial_box>
-    </link>
-    <link name="right_fork">
-        <visual>
-            <origin xyz="0.575 0 0.025"/>
-            <geometry>
-                <box size="1.15 0.14 0.05"/>
-            </geometry>
-            <material name="white"/>
-        </visual>
-        <collision>
-            <origin xyz="0.575 0 0.025"/>
-            <geometry>
-                <box size="1.15 0.14 0.05"/>
-            </geometry>
-            <material name="white"/>
-        </collision>
-        <xacro:inertial_box mass="5.0" x="1.14" y="0.14" z="0.05">
-            <origin xyz="0.575 0 0.025" rpy="0 0 0"/>
-        </xacro:inertial_box>
+        </xacro:inertial_sphere>
     </link>
     <!-- Bağlantılar -->
-    <joint name="fork_left_wheel_joint" type="continuous">
+    <joint name="left_wheel_joint" type="continuous">
         <parent link="base_link"/>
-        <child link="fork_left_wheel"/>
-        <origin xyz="-0.94 0.18 -0.05" rpy="-${pi/2} 0 0" />
+        <child link="left_wheel"/>
+        <origin xyz="-0.0 0.055 -0.05" rpy="-${pi/2} 0 0" />
         <axis xyz="0 0 1"/>
     </joint>
-    <joint name="fork_right_wheel_joint" type="continuous">
+    <joint name="right_wheel_joint" type="continuous">
         <parent link="base_link"/>
-        <child link="fork_right_wheel"/>
-        <origin xyz="-0.94 -0.18 -0.05" rpy="-${pi/2} 0 0" />
+        <child link="right_wheel"/>
+        <origin xyz="-0.0 -0.055 -0.05" rpy="-${pi/2} 0 0" />
         <axis xyz="0 0 -1"/>
     </joint>
-    <joint name="front_wheel_joint" type="continuous">
-        <parent link="steering_cylinder"/>
-        <child link="front_wheel"/>
-        <origin xyz="0.0 0.0 -0.1" rpy="0 -${3*pi/2} 0" /> <!--origin xyz="0.0 0.0 -0.1" rpy="0 ${3*pi/2} 0" /-->
-        <axis xyz="0 0 1"/>
-    </joint>
-    <joint name="steering_cylinder_joint" type="revolute">
+    <joint name="caster_wheel_joint" type="fixed">
         <parent link="base_link"/>
-        <child link="steering_cylinder"/>
-        <origin xyz="0.0 0.0 0.1" rpy="0 0 ${pi/2}" />
+        <child link="caster_wheel"/>
+        <origin xyz="0.07 -0.0 -0.05" rpy="-${pi/2} 0 0" />
         <axis xyz="0 0 -1"/>
-        <limit effort="10.0" velocity="1.0" lower="-0.872664626" upper="0.872664626"/>
-    </joint>
-    <joint name="left_fork_joint" type="fixed">
-        <parent link="base_link"/>
-        <child link="left_fork"/>
-        <origin xyz="-1.15 0.18 -0.05"/>
-    </joint>
-    <joint name="right_fork_joint" type="fixed">
-        <parent link="base_link"/>
-        <child link="right_fork"/>
-        <origin xyz="-1.15 -0.18 -0.05"/>
     </joint>
 </robot>
