Commit message: slam & navigation sim update

File: description/lidar.xacro (robot description, xacro)
@@ -26,19 +26,19 @@
     <gazebo reference="laser">
       <material value="Gazebo/Blue"/>
-      <sensor type="gpu_lidar" name="head_hokuyo_sensor">
-        <pose>0.075 0.0 0.0125 0 0 0</pose>
+      <sensor type="gpu_lidar" name="slamtec_C1">
+        <pose>0.0 0.0 0.052375 0 0 0</pose>
         <visualize>false</visualize>
-        <update_rate>10</update_rate>
+        <update_rate>50</update_rate>
         <lidar>
           <scan>
             <horizontal>
-              <samples>270</samples>
-              <min_angle>-2.0943</min_angle>
-              <max_angle>2.0943</max_angle>
+              <samples>5000</samples>
+              <min_angle>-3.1415926536</min_angle>
+              <max_angle>3.1415926536</max_angle>
             </horizontal>
           </scan>
           <range>
-            <min>0.10</min>
-            <max>20.0</max>
+            <min>0.05</min>
+            <max>12.0</max>
           </range>
         </lidar>

File: description/robot_model.xacro (robot description, xacro)
@@ -100,5 +100,5 @@
         <parent link="base_link"/>
         <child link="left_wheel"/>
-        <origin xyz="-0.02 0.055 -0.0325" rpy="-${pi/2} 0 0" />
+        <origin xyz="0.0 0.055 -0.0325" rpy="-${pi/2} 0 0" />
         <axis xyz="0 0 1"/>
     </joint>
@@ -106,5 +106,5 @@
         <parent link="base_link"/>
         <child link="right_wheel"/>
-        <origin xyz="-0.02 -0.055 -0.0325" rpy="-${pi/2} 0 0" />
+        <origin xyz="0.0 -0.055 -0.0325" rpy="-${pi/2} 0 0" />
         <axis xyz="0 0 1"/>
     </joint>

Commit message: hardware interface

File: description/lidar.xacro (robot description, xacro)
@@ -2,5 +2,5 @@
 <robot xmlns:xacro="http://ros.org/wiki/xacro">
     <joint name="laser_joint" type="fixed">
-      <origin xyz="0.0 0.0 0.052375" rpy="0 0 0"/>
+      <origin xyz="0.0 0.0 0.052375" rpy="0 0 ${pi}"/>
       <parent link="base_link"/>
       <child link="laser"/>

File: description/robot.urdf.xacro (robot description, xacro)
@@ -3,4 +3,5 @@
     <xacro:include filename="robot_model.xacro" />
     <xacro:include filename="lidar.xacro" />
-    <xacro:include filename="gz_control.xacro" />
+    <!--xacro:include filename="gz_control.xacro" /-->
+    <xacro:include filename="robot_control.xacro" />
 </robot>

File: description/robot_control.xacro (robot description, xacro)
@@ -1,17 +1,22 @@
-<ros2_control name="DiffDriveControl" type="system">
-    <hardware>
-      <plugin>diff_robot/DiffBotSystemHardware</plugin>
-      <param name="device">/dev/ttyUSB0</param>
-      <param name="baud_rate">115200</param>
-    </hardware>
-    <joint name="left_wheel_joint">
-      <command_interface name="velocity"/>
-      <state_interface name="position"/>
-      <state_interface name="velocity"/>
-    </joint>
-    <joint name="right_wheel_joint">
-      <command_interface name="velocity"/>
-      <state_interface name="position"/>
-      <state_interface name="velocity"/>
-    </joint>
-</ros2_control>
+<?xml version="1.0"?>
+<robot xmlns:xacro="http://www.ros.org/wiki/xacro">
+  <ros2_control name="DiffDriveControl" type="system">
+      <hardware>
+        <plugin>diff_robot/DiffBotSystemHardware</plugin>
+        <param name="left_wheel_joint">left_wheel_joint</param>
+        <param name="right_wheel_joint">right_wheel_joint</param>
+        <param name="device">/dev/ttyUSB1</param>
+        <param name="baud_rate">115200</param>
+      </hardware>
+      <joint name="left_wheel_joint">
+        <command_interface name="velocity"/>
+        <state_interface name="position"/>
+        <state_interface name="velocity"/>
+      </joint>
+      <joint name="right_wheel_joint">
+        <command_interface name="velocity"/>
+        <state_interface name="position"/>
+        <state_interface name="velocity"/>
+      </joint>
+  </ros2_control>
+</robot>
