Commit message: ros2_control & gazebo done

File: description/robot.urdf.xacro (robot description, xacro)
@@ -3,3 +3,4 @@
     <xacro:include filename="robot_model.xacro" />
     <xacro:include filename="lidar.xacro" />
+    <xacro:include filename="gz_control.xacro" />
 </robot>

File: description/robot_model.xacro (robot description, xacro)
@@ -19,6 +19,6 @@
     <!-- BASE_FOOTPRINT LINK-->
     <joint name="base_footprint_joint" type="fixed">
-        <parent link="base_footprint"/>
-        <child link="base_link"/>
+        <parent link="base_link"/>
+        <child link="base_footprint"/>
         <origin xyz="0 0 0" rpy="0 0 0"/>
     </joint>
@@ -88,9 +88,9 @@
         <collision>
             <geometry>
-                <sphere radius="0.05"/>
+                <sphere radius="0.015"/>
             </geometry>
             <material name="red"/>
         </collision>
-        <xacro:inertial_sphere mass="0.15" radius="0.05">
+        <xacro:inertial_sphere mass="0.15" radius="0.015">
             <origin xyz="0 0 0" rpy="0 0 0"/>
         </xacro:inertial_sphere>
@@ -100,5 +100,5 @@
         <parent link="base_link"/>
         <child link="left_wheel"/>
-        <origin xyz="-0.0 0.055 -0.05" rpy="-${pi/2} 0 0" />
+        <origin xyz="-0.02 0.055 -0.0325" rpy="-${pi/2} 0 0" />
         <axis xyz="0 0 1"/>
     </joint>
@@ -106,12 +106,12 @@
         <parent link="base_link"/>
         <child link="right_wheel"/>
-        <origin xyz="-0.0 -0.055 -0.05" rpy="-${pi/2} 0 0" />
-        <axis xyz="0 0 -1"/>
+        <origin xyz="-0.02 -0.055 -0.0325" rpy="-${pi/2} 0 0" />
+        <axis xyz="0 0 1"/>
     </joint>
     <joint name="caster_wheel_joint" type="fixed">
         <parent link="base_link"/>
         <child link="caster_wheel"/>
-        <origin xyz="0.07 -0.0 -0.05" rpy="-${pi/2} 0 0" />
-        <axis xyz="0 0 -1"/>
+        <origin xyz="0.07 0.0 -0.05" rpy="0 0 0" />
+        <axis xyz="0 0 1"/>
     </joint>
 </robot>

Commit message: description update

File: description/robot.urdf.xacro (robot description, xacro)
@@ -1,7 +1,7 @@
 <?xml version="1.0"?>
 <robot xmlns:xacro="http://www.ros.org/wiki/xacro"  name="robot">
-    <xacro:include filename="robot_model.xacro" />
+    <xacro:include filename="robot_model2.xacro" />
     <xacro:include filename="lidar.xacro" />
-    <!--xacro:include filename="gz_control.xacro" /-->
-    <xacro:include filename="robot_control.xacro" />
+    <xacro:include filename="gz_control.xacro" />
+    <!--xacro:include filename="robot_control.xacro" /-->
 </robot>

File: description/robot_model2.xacro (robot description, xacro)
@@ -29,5 +29,5 @@
             <origin xyz="0.0 0.0 0.0" rpy="0 0 0"/>
             <geometry>
-                <box size="0.17386 0.140 0.080"/>
+                <box size="0.175 0.110 0.07975"/>
             </geometry>
             <material name="black"/>
@@ -36,9 +36,9 @@
             <origin xyz="0.0 0.0 0.0" rpy="0 0 0"/>
             <geometry>
-                <box size="0.17386 0.140 0.080"/>
+                <box size="0.175 0.110 0.07975"/>
             </geometry>
             <material name="black"/>
         </collision>
-        <xacro:inertial_box mass="0.5" x="0.17386" y="0.140" z="0.080">
+        <xacro:inertial_box mass="0.5" x="0.175" y="0.110" z="0.07975">
             <origin xyz="0.0 0.0 0.0" rpy="0 0 0"/>
         </xacro:inertial_box>
@@ -48,5 +48,5 @@
         <visual>
             <geometry>
-                <cylinder radius="0.03" length="0.03"/>
+                <cylinder radius="0.0325" length="0.03"/>
             </geometry>
             <material name="orange"/>
@@ -54,9 +54,9 @@
         <collision>
             <geometry>
-                <cylinder radius="0.03" length="0.03"/>
+                <cylinder radius="0.0325" length="0.03"/>
             </geometry>
             <material name="orange"/>
         </collision>
-        <xacro:inertial_cylinder mass="0.01" length="0.03" radius="0.03">
+        <xacro:inertial_cylinder mass="0.1" length="0.03" radius="0.0325">
             <origin xyz="0 0 0" rpy="0 0 0"/>
         </xacro:inertial_cylinder>
@@ -65,5 +65,5 @@
         <visual>
             <geometry>
-                <cylinder radius="0.03" length="0.03"/>
+                <cylinder radius="0.0325" length="0.03"/>
             </geometry>
             <material name="orange"/>
@@ -71,9 +71,9 @@
         <collision>
             <geometry>
-                <cylinder radius="0.03" length="0.03"/>
+                <cylinder radius="0.0325" length="0.03"/>
             </geometry>
             <material name="orange"/>
         </collision>
-        <xacro:inertial_cylinder mass="0.01" length="0.03" radius="0.03">
+        <xacro:inertial_cylinder mass="0.1" length="0.03" radius="0.0325">
             <origin xyz="0 0 0" rpy="0 0 0"/>
         </xacro:inertial_cylinder>
@@ -82,5 +82,5 @@
         <visual>
             <geometry>
-                <sphere radius="0.01" />
+                <sphere radius="0.015" />
             </geometry>
             <material name="red"/>
@@ -88,9 +88,9 @@
         <collision>
             <geometry>
-                <sphere radius="0.01"/>
+                <sphere radius="0.015"/>
             </geometry>
             <material name="red"/>
         </collision>
-        <xacro:inertial_sphere mass="0.01" radius="0.01">
+        <xacro:inertial_sphere mass="0.15" radius="0.015">
             <origin xyz="0 0 0" rpy="0 0 0"/>
         </xacro:inertial_sphere>
@@ -100,5 +100,5 @@
         <parent link="base_link"/>
         <child link="left_wheel"/>
-        <origin xyz="-0.08693 0.085 -0.0325" rpy="-${pi/2} 0 0" />
+        <origin xyz="0.0 0.055 -0.0325" rpy="-${pi/2} 0 0" />
         <axis xyz="0 0 1"/>
     </joint>
@@ -106,5 +106,5 @@
         <parent link="base_link"/>
         <child link="right_wheel"/>
-        <origin xyz="-0.08693 -0.085 -0.0325" rpy="-${pi/2} 0 0" />
+        <origin xyz="0.0 -0.055 -0.0325" rpy="-${pi/2} 0 0" />
         <axis xyz="0 0 1"/>
     </joint>
@@ -112,5 +112,5 @@
         <parent link="base_link"/>
         <child link="caster_wheel"/>
-        <origin xyz="0.02193 0.0 -0.05" rpy="0 0 0" />
+        <origin xyz="0.07 0.0 -0.05" rpy="0 0 0" />
         <axis xyz="0 0 1"/>
     </joint>
